File: STM32WB55_QFN48_IPD_REF_BOARD.kicad_pcb (KiCad board)
At the start: 4 copper layers, 72 parts, among them IC1 LD3985M33R, IC2 USBLC6-2SC6, J1 USB_B_Micro, J2 Conn_01x05_Male, J3 Conn_01x02_Male, J4 Conn_01x04_Male, J5 Conn_01x01_Male, J6 Conn_01x01_Male, J7 Conn_01x08_Male, U1 MCP1640CCH, U2 STM32WB55CG, U4 BNO055_my, U5 ADS1115IDGS, Y1 NX2520SA-32MHz, Y2 NX2012SA-32768K, Y3 NX2012SA-32768K

Commit message: v01
Parts:
- removed J3: Conn_01x02_Male, 0Pretty:pin_02
- removed J6: Conn_01x01_Male, 0Pretty:pin_01
- removed U1: MCP1640CCH, Package_TO_SOT_SMD:SOT-23-6
- added I2C: Conn_01x02_Male, 0Pretty:pin_02, F.Cu at (137.3, 113.6)
- added MCP: MCP1640CCH, Package_TO_SOT_SMD:SOT-23-6, F.Cu at (91.0, 105.2)
- added N1: Housing, Symbol:KiCad-Logo2_5mm_Copper, B.Cu at (153.9, 109.8)
- added NRSTR: Conn_01x01_Male, 0Pretty:pin_01, F.Cu at (125.3, 113.5)
- J7: moved to B.Cu
- U2: value STM32WB55CG -> STM32
- moved R7 3.54 mm to (130.7, 106.8), turned to 180 degrees
- moved R8 2.86 mm to (131.8, 105.3), turned to 90 degrees
- moved R13 2.52 mm to (134.5, 108.5)
- moved C20 2.49 mm to (129.4, 108.0)
- moved FB2 2.43 mm to (130.7, 108.5)
- moved C_1 2.28 mm to (89.2, 107.1)
- moved C22 2.28 mm to (130.7, 107.7)
- moved R_1 2.22 mm to (92.7, 107.1), turned to 0 degrees
- moved J4 2.10 mm to (133.2, 103.8)
- moved FB3 1.99 mm to (134.0, 105.4)
- moved BT1 1.89 mm to (91.7, 102.7)
- moved U5 1.85 mm to (132.6, 107.4)
- moved J1 1.77 mm to (79.4, 107.0)
- moved R9 1.77 mm to (133.2, 105.3), turned to 90 degrees
- moved R_2 1.76 mm to (93.2, 105.1)
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- renumbered Y2 to 32768K, Y1 to 32MHz, ed1 to Coax
Connections:
- U2 pad 49: (no net) -> GND
Routing:
- net GND: track 105.9 -> 69.7 mm, vias 31 -> 29
- net 3v3fromUSB: track 18.3 -> 0.00 mm, vias 2 -> 1
- net Net-(D3-Pad2): track 16.1 -> 1.13 mm
- net USB_D-: track 24.3 -> 12.2 mm
- net USB_D+: track 21.5 -> 12.0 mm
- net +5V: track 11.1 -> 3.40 mm
- net +3V3: track 36.7 -> 29.3 mm, vias 13 -> 19
- net Net-(J4-Pad4): track 0.00 -> 4.60 mm
- net Net-(J4-Pad3): track 0.00 -> 4.57 mm
- net Net-(J4-Pad2): track 0.00 -> 4.24 mm
- net USB_OD-: track 5.35 -> 2.17 mm
- net USB_OD+: track 7.93 -> 4.94 mm
- net 3v3fromBAT: track 11.6 -> 9.53 mm, vias 3 -> 2
- net Net-(FB3-Pad1): track 0.00 -> 1.87 mm
- net Net-(C14-Pad1): track 1.85 -> 0.00 mm
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Other:
- net class +3.3V added: clearance 0.2, trace_width 0.25, via_dia 0.5, via_drill 0.4
- net class GND added: clearance 0.2, trace_width 0.25, via_dia 0.5, via_drill 0.3
- net class USB Data added: clearance 0.2, trace_width 0.25, via_dia 0.8, via_drill 0.4
- board text added: "+"

Commit message: v02
Parts:
- removed 32768K: NX2012SA-32768K, 0Pretty:Crystal_2012_custom
- removed 32MHz: NX2520SA-32MHz, Crystal:Crystal_SMD_2520-4Pin_2.5x2.0mm
- removed Coax: RECE.20279.001E.01, RECE_antena_connector:RECE.20279.001E.01
- removed I2C: Conn_01x02_Male, 0Pretty:pin_02
- removed J2: Conn_01x05_Male, 0Pretty:pin_03
- removed J7: Conn_01x08_Male, 0Pretty:pin_08
- removed MCP: MCP1640CCH, Package_TO_SOT_SMD:SOT-23-6
- removed NRSTR: Conn_01x01_Male, 0Pretty:pin_01
- removed S2: MLL1200S, vypinac:MLL1200S
- removed U4: BNO055_my, Package_LGA:LGA-28_5.2x3.8mm_P0.5mm
- removed U5: ADS1115IDGS, ADS1115:ADS1115IRUGR
- added ADS1115: ADS1115IDGS, ADS1115:ADS1115IRUGR, F.Cu at (135.8, 89.2)
- added BNO55: BNO055_my, Package_LGA:LGA-28_5.2x3.8mm_P0.5mm, F.Cu at (174.5, 90.4)
- added J_GEN1: Conn_01x03_Male, 0Pretty:pin_03, B.Cu at (102.4, 84.7)
- added J_GND1: Conn_01x01_Male, 0Pretty:pin_01, B.Cu at (79.4, 87.4)
- added J_I2C1: Conn_01x02_Male, 0Pretty:pin_02, F.Cu at (136.2, 96.2)
- added J_NRST1: Conn_01x01_Male, 0Pretty:pin_01, F.Cu at (95.8, 96.3)
- added J_PWR1: Conn_01x01_Male, 0Pretty:pin_01, B.Cu at (79.4, 92.5)
- added J_SPI1: Conn_01x03_Male, 0Pretty:pin_03, F.Cu at (130.2, 96.2)
- added J_SWD1: Conn_01x03_Male, 0Pretty:pin_03, B.Cu at (92.5, 96.3)
- added MCP1640: MCP1640CCH, Package_TO_SOT_SMD:SOT-23-6, F.Cu at (94.7, 87.8)
- added S_PWR1: MLL1200S, vypinac:MLL1200S, B.Cu at (87.3, 85.6)
- added Y1: NX2520SA-32MHz, Crystal:Crystal_SMD_2520-4Pin_2.5x2.0mm, F.Cu at (113.5, 85.7)
- added Y2: NX2012SA-32768K, 0Pretty:Crystal_2012_custom, F.Cu at (104.5, 96.3)
- added ed1: RECE.20279.001E.01, RECE_antena_connector:RECE.20279.001E.01, F.Cu at (119.6, 85.8)
- U2: value STM32 -> STM32WB55CG
- moved D2 30.8 mm to (97.7, 96.3), turned to 270 degrees
- moved R5 27.8 mm to (99.2, 96.6), turned to 270 degrees
- moved C19 26.1 mm to (100.2, 96.6), turned to 90 degrees
- moved R2 23.7 mm to (139.8, 94.3), turned to 90 degrees
- moved R3 22.1 mm to (138.8, 94.3), turned to 90 degrees
- moved S_BOOT1 22.1 mm to (122.2, 96.2), turned to 180 degrees
- moved N1 19.2 mm to (156.5, 90.8), turned to 180 degrees
- moved R7 18.7 mm to (133.4, 88.3)
- moved R12 18.6 mm to (138.4, 88.9)
- moved C22 18.6 mm to (133.7, 89.3)
- moved FB3 18.6 mm to (137.3, 87.2)
- moved J4 18.5 mm to (136.4, 85.5)
- moved R8 18.5 mm to (135.0, 87.0)
- moved R9 18.5 mm to (136.4, 87.0)
- moved C20 18.4 mm to (132.2, 89.8)
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- renumbered J5 to J_BNO055RST1, S1 to S_BOOT1
Connections:
- FL1 pad 1: Net-(FL1-Pad1) -> /R_OUT
Routing:
- net I2C_SCL: track 2.00 -> 83.7 mm, vias 1 -> 3
- net BNO055_INT: track 2.09 -> 82.9 mm
- net I2C_SDA: track 3.61 -> 82.7 mm, vias 1 -> 2
- net ADC_ALERT: track 1.76 -> 42.5 mm
- net +3V3: track 29.3 -> 68.9 mm, vias 19 -> 33
- net SPI_MOSI: track 1.04 -> 25.5 mm
- net SPI_MISO: track 1.00 -> 21.0 mm
- net SPI_SCK: track 1.12 -> 19.7 mm
- net Net-(R4-Pad1): track 2.38 -> 20.4 mm, vias 1 -> 3
- net Net-(C19-Pad1): track 0.00 -> 16.8 mm
- net Net-(BNO55-Pad11): track 1.13 -> 14.5 mm
- net USB_D-: track 12.2 -> 23.2 mm
- net 3v3fromBAT: track 9.53 -> 19.1 mm
- net 3v3fromUSB: track 0.00 -> 8.64 mm, vias 1 -> 2
- net USB_D+: track 12.0 -> 20.5 mm
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- added copper zone on PWD, net +3V3
- added copper zone on B.Cu, net GND
- added copper zone on F.Cu, net GND
- added copper zone on GND, net GND
Other:
- board outline added: 99.4 x 14.3 mm
- net class +3.3V: clearance 0.2 -> 0.1
- net class Default: clearance 0.2 -> 0.1
- net class GND: clearance 0.2 -> 0.1; trace_width 0.25 -> 0.2
- net class I2C added: clearance 0.2, trace_width 0.277, via_dia 0.8, via_drill 0.4
- net class RF added: clearance 0.11, trace_width 0.2, via_dia 0.8, via_drill 0.4
- net class RF_OUT added: clearance 0.127, trace_width 0.45, via_dia 0.8, via_drill 0.4
- rule trace_clearance: 0.2 -> 0.1

Commit message: v03
Parts:
- removed IC1: LD3985M33R, Package_TO_SOT_SMD:SOT-23-5
- removed S_BOOT1: MLL1200S, vypinac:MLL1200S
- added BOOT: MLL1200S, vypinac:MLL1200S, B.Cu at (122.2, 96.2)
- added LD3985M33R: LD3985M33R, Package_TO_SOT_SMD:SOT-23-5, F.Cu at (88.2, 87.8)
- added REF**: FIT_napis, 0Pretty:FIT_napis, F.Cu at (152.3, 93.3)
- N1: moved to F.Cu
- moved SWD 3.50 mm to (89.0, 96.3)
- moved C19 3.20 mm to (97.0, 96.6)
- moved D2 3.20 mm to (94.5, 96.3)
- moved NRST 3.20 mm to (92.5, 96.3)
- moved R5 3.20 mm to (96.0, 96.6)
- moved C1 0.98 mm to (116.0, 87.6)
- moved C2 0.98 mm to (116.0, 86.6)
- moved J_SPI1 0.30 mm to (130.6, 96.2)
- renumbered Y1 to 32MHz, J_BNO055RST1 to BNO055RST, Y2 to CLK, J_GND1 to GND, J_I2C1 to I2C, J_NRST1 to NRST, J_PWR1 to PWR, J_SWD1 to SWD, S_PWR1 to S_PWR, IC2 to USBLC6-2SC6
Routing:
- net SYS_JTMS-SWDIO: track 18.2 -> 21.7 mm
- net SYS_JTDO-SWO: track 12.6 -> 16.1 mm
- net SYS_JTCK-SWCLK: track 16.1 -> 19.6 mm
- net Net-(C19-Pad1): track 16.8 -> 20.0 mm
- net +3V3: track 68.9 -> 68.4 mm
- net /R_OUT: track 6.63 -> 6.10 mm
- net GND: vias 38 -> 35
